File: kicad/rpi-balatro-board/rpi-balatro-board.kicad_sch (KiCad schematic)
At the start: 43 parts, among them J1 Raspberry_Pi_4, J2 Conn_01x01_Socket, J3 Conn_01x01_Socket, J4 Conn_01x01_Socket, J5 Conn_01x01_Socket, J6 Conn_01x01_Socket, M1 RFID-RC522, M2 RFID-RC522, M3 RFID-RC522, M4 RFID-RC522, M5 RFID-RC522, M6 RFID-RC522, SW1 SW_Push, SW10 SW_Push, SW11 SW_Push, SW12 SW_Push, SW13 SW_Push, SW2 SW_Push, SW3 SW_Push, SW4 SW_Push, SW5 SW_Push, SW6 SW_Push, SW7 SW_Push, SW8 SW_Push, SW9 SW_Push, U1 MAX7221xNG, U2 74HC595, U3 MAX7221xNG

Commit message: polly ollu
Connections:
- net at J1.1 (3V3), J1.17 (3V3): now also M1.8 (3V3), M2.8 (3V3), M3.8 (3V3), M4.8 (3V3), M5.8 (3V3), M6.8 (3V3), U2.16 (VCC)
- net at J1.14 (GND), J1.20 (GND), J1.25 (GND)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: now also M1.6 (GND)
- net at J1.19 (MOSI_SPI0/GPIO10), U1.1 (DIN): now also M2.3 (MOSI), M3.3 (MOSI), M4.3 (MOSI), M5.3 (MOSI), M6.3 (MOSI)
- net at J1.21 (MISO_SPI0/GPIO09): now also M1.3 (MOSI), M1.4 (MISO), M2.4 (MISO), M3.4 (MISO), M4.4 (MISO), M5.4 (MISO), M6.4 (MISO)
- net at J1.23 (SCLK_SPI0/GPIO11), U1.13 (CLK), U3.13 (CLK): now also M1.2 (SCK), M2.2 (SCK), M3.2 (SCK), M4.2 (SCK), M5.2 (SCK), M6.2 (SCK)
- net at SW2.1: now also J4.1 (Pin_1), SW1.1, SW11.1, SW12.1
