File: kicad/rpi-balatro-board/rpi-balatro-board.kicad_sch (KiCad schematic)
At the start: 58 parts, among them J1 Conn_01x01_Socket, J2 Conn_01x01_Socket, J3 Conn_01x01_Socket, J4 Conn_01x01_Socket, J5 Conn_01x01_Socket, J6 Conn_01x01_Socket, J7 Conn_01x01_Socket, M1 RFID-RC522, M2 RFID-RC522, M3 RFID-RC522, M4 RFID-RC522, M5 RFID-RC522, M6 RFID-RC522, SW1 SW_Push, SW10 SW_Push, SW11 SW_Push, SW12 SW_Push, SW13 SW_Push, SW2 SW_Push, SW3 SW_Push, SW4 SW_Push, SW5 SW_Push, SW6 SW_Push, SW7 SW_Push, SW8 SW_Push, SW9 SW_Push, U1 MAX7221xNG, U2 MAX7221xNG, U3 74HC595

Commit message: addicted to pla
Other:
- sheet digit_max_2: file dig_max_1.kicad_sch -> dig_max_2.kicad_sch
Changed lines of the file:
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@@
 			)
 		)
-		(property "Sheetfile" "dig_max_1.kicad_sch"
+		(property "Sheetfile" "dig_max_2.kicad_sch"
 			(at 123.7746 118.11 90)
 			(effects
