File: kicad/rpi-balatro-board/dig_max_1.kicad_sch (KiCad schematic)
At the start: 8 parts, among them U11 SM420561N, U12 SM420561N, U13 SM420561N, U14 SM420561N, U15 SM420561N, U16 SM420561N, U17 SM420561N, U18 SM420561N

Commit message: botbotbot
Parts:
- removed U17, U18: SM420561N, Display_7Segment:7SegmentLED_LTS6760_LTS6780, symbol Display_Character:SM420561N

Commit message: addicted to pla
Parts:
- added U17, U18: SM420561N, Display_7Segment:7SegmentLED_LTS6760_LTS6780, symbol Display_Character:SM420561N
Connections:
- net SEG_A: now also U17.7 (A), U18.7 (A)
- net SEG_B: now also U17.6 (B), U18.6 (B)
- net SEG_C: now also U17.4 (C), U18.4 (C)
- net SEG_D: now also U17.2 (D), U18.2 (D)
- net SEG_DP: now also U17.5 (DP), U18.5 (DP)
- net SEG_E: now also U17.1 (E), U18.1 (E)
- net SEG_F: now also U17.9 (F), U18.9 (F)
- net SEG_G: now also U17.10 (G), U18.10 (G)
- new net DIG_6: U17.8 (CC)
- new net DIG_7: U18.8 (CC)
