File: kicad/rpi-balatro-board/rpi-balatro-board.kicad_pcb (KiCad board)
At the start: 2 copper layers, 21 parts, among them J1 Raspberry_Pi_4, U1 MAX7221xNG, U11 SM420561N, U12 SM420561N, U13 SM420561N, U14 SM420561N, U15 SM420561N, U16 SM420561N, U17 SM420561N, U18 SM420561N, U19 SM420561N, U20 SM420561N, U21 SM420561N, U22 SM420561N, U23 SM420561N, U24 SM420561N, U25 SM420561N, U26 SM420561N, U3 MAX7221xNG

Commit message: botbotbot
Parts:
- removed U17, U18: SM420561N, Display_7Segment:7SegmentLED_LTS6760_LTS6780
- added 3V1: Conn_01x01_Socket, Connector_PinHeader_2.54mm:PinHeader_1x01_P2.54mm_Vertical, B.Cu at (190.5, 93.0)
- added 5V1: Conn_01x01_Socket, Connector_PinHeader_2.54mm:PinHeader_1x01_P2.54mm_Vertical, B.Cu at (83.5, 52.0)
- added B1: Conn_01x01_Socket, Connector_PinHeader_2.54mm:PinHeader_1x01_P2.54mm_Vertical, B.Cu at (67.5, 143.6)
- added B2: Conn_01x01_Socket, Connector_PinHeader_2.54mm:PinHeader_1x01_P2.54mm_Vertical, B.Cu at (294.5, 135.8)
- added B3: Conn_01x01_Socket, Connector_PinHeader_2.54mm:PinHeader_1x01_P2.54mm_Vertical, B.Cu at (132.5, 188.3)
- added B4: Conn_01x01_Socket, Connector_PinHeader_2.54mm:PinHeader_1x01_P2.54mm_Vertical, B.Cu at (190.0, 134.8)
- added D1: 1N914, Diode_THT:D_DO-35_SOD27_P7.62mm_Horizontal, B.Cu at (202.0, 134.8)
- added D10: 1N914, Diode_THT:D_DO-35_SOD27_P7.62mm_Horizontal, B.Cu at (151.0, 188.3)
- added D11: 1N914, Diode_THT:D_DO-35_SOD27_P7.62mm_Horizontal, B.Cu at (312.0, 135.8)
- added D12: 1N914, Diode_THT:D_DO-35_SOD27_P7.62mm_Horizontal, B.Cu at (86.3, 143.6)
- added D13: 1N914, Diode_THT:D_DO-35_SOD27_P7.62mm_Horizontal, B.Cu at (78.4, 143.6)
- added D2: 1N914, Diode_THT:D_DO-35_SOD27_P7.62mm_Horizontal, B.Cu at (146.0, 188.3)
- added D3: 1N914, Diode_THT:D_DO-35_SOD27_P7.62mm_Horizontal, B.Cu at (83.6, 143.6)
- added D4: 1N914, Diode_THT:D_DO-35_SOD27_P7.62mm_Horizontal, B.Cu at (309.5, 135.8)
- added D5: 1N914, Diode_THT:D_DO-35_SOD27_P7.62mm_Horizontal, B.Cu at (81.0, 143.6)
- added D6: 1N914, Diode_THT:D_DO-35_SOD27_P7.62mm_Horizontal, B.Cu at (148.5, 188.3)
- added D7: 1N914, Diode_THT:D_DO-35_SOD27_P7.62mm_Horizontal, B.Cu at (307.0, 135.8)
- added D8: 1N914, Diode_THT:D_DO-35_SOD27_P7.62mm_Horizontal, B.Cu at (207.0, 134.8)
- added D9: 1N914, Diode_THT:D_DO-35_SOD27_P7.62mm_Horizontal, B.Cu at (204.5, 134.8)
- added GND1: Conn_01x01_Socket, Connector_PinHeader_2.54mm:PinHeader_1x01_P2.54mm_Vertical, B.Cu at (166.0, 72.0)
- added IRQ1: Conn_01x01_Socket, Connector_PinHeader_2.54mm:PinHeader_1x01_P2.54mm_Vertical, B.Cu at (16.3, 24.4)
- added J2: Conn_01x01_Socket, Connector_PinHeader_2.54mm:PinHeader_1x01_P2.54mm_Vertical, B.Cu at (79.0, 77.5)
- added J3: Conn_01x01_Socket, Connector_PinHeader_2.54mm:PinHeader_1x01_P2.54mm_Vertical, B.Cu at (86.0, 77.5)
- added J4: Conn_01x01_Socket, Connector_PinHeader_2.54mm:PinHeader_1x01_P2.54mm_Vertical, B.Cu at (244.5, 130.5)
- added J5: Conn_01x01_Socket, Connector_PinHeader_2.54mm:PinHeader_1x01_P2.54mm_Vertical, B.Cu at (33.0, 109.5)
- added J6: Conn_01x01_Socket, Connector_PinHeader_2.54mm:PinHeader_1x01_P2.54mm_Vertical, B.Cu at (260.0, 107.5)
- added J7: Conn_01x01_Socket, Connector_PinHeader_2.54mm:PinHeader_1x01_P2.54mm_Vertical, B.Cu at (195.5, 99.3)
- added M1: RFID-RC522, RFID-RC522:RFID-RC522, F.Cu at (257.5, 206.1)
- added M2: RFID-RC522, RFID-RC522:RFID-RC522, F.Cu at (327.5, 206.1)
- added M3: RFID-RC522, RFID-RC522:RFID-RC522, F.Cu at (117.5, 206.1)
- added M4: RFID-RC522, RFID-RC522:RFID-RC522, F.Cu at (187.5, 88.6)
- added M5: RFID-RC522, RFID-RC522:RFID-RC522, F.Cu at (187.5, 206.1)
- added M6: RFID-RC522, RFID-RC522:RFID-RC522, F.Cu at (47.5, 206.1)
- added MAXCS1: Conn_01x01_Socket, Connector_PinHeader_2.54mm:PinHeader_1x01_P2.54mm_Vertical, B.Cu at (16.3, 29.0)
- added MISO1: Conn_01x01_Socket, Connector_PinHeader_2.54mm:PinHeader_1x01_P2.54mm_Vertical, B.Cu at (16.3, 33.6)
- added MOSI1: Conn_01x01_Socket, Connector_PinHeader_2.54mm:PinHeader_1x01_P2.54mm_Vertical, B.Cu at (20.9, 38.5)
- added RST1: Conn_01x01_Socket, Connector_PinHeader_2.54mm:PinHeader_1x01_P2.54mm_Vertical, B.Cu at (20.9, 43.1)
- added SCK1: Conn_01x01_Socket, Connector_PinHeader_2.54mm:PinHeader_1x01_P2.54mm_Vertical, B.Cu at (16.3, 38.5)
- added SCS1: Conn_01x01_Socket, Connector_PinHeader_2.54mm:PinHeader_1x01_P2.54mm_Vertical, B.Cu at (16.3, 43.1)
- added SW1: SW_Push, Button_Switch_Keyboard:SW_Cherry_MX_1.00u_PCB, F.Cu at (173.0, 113.4)
- added SW10: SW_Push, Button_Switch_Keyboard:SW_Cherry_MX_1.00u_PCB, F.Cu at (207.0, 113.4)
- added SW11: SW_Push, Button_Switch_Keyboard:SW_Cherry_MX_1.00u_PCB, F.Cu at (137.0, 113.4)
- added SW12: SW_Push, Button_Switch_Keyboard:SW_Cherry_MX_1.00u_PCB, F.Cu at (347.8, 113.9)
- added SW13: SW_Push, Button_Switch_Keyboard:SW_Cherry_MX_1.00u_PCB, F.Cu at (33.0, 113.4)
- added SW2: SW_Push, Button_Switch_Keyboard:SW_Cherry_MX_1.00u_PCB, F.Cu at (143.1, 72.9)
- added SW3: SW_Push, Button_Switch_Keyboard:SW_Cherry_MX_1.00u_PCB, F.Cu at (103.0, 113.4)
- added SW4: SW_Push, Button_Switch_Keyboard:SW_Cherry_MX_1.00u_PCB, F.Cu at (312.0, 113.4)
- added SW5: SW_Push, Button_Switch_Keyboard:SW_Cherry_MX_1.00u_PCB, F.Cu at (67.0, 113.4)
- added SW6: SW_Push, Button_Switch_Keyboard:SW_Cherry_MX_1.00u_PCB, F.Cu at (277.0, 113.4)
- added SW7: SW_Push, Button_Switch_Keyboard:SW_Cherry_MX_1.00u_PCB, F.Cu at (157.4, 234.1)
- added SW8: SW_Push, Button_Switch_Keyboard:SW_Cherry_MX_1.00u_PCB, F.Cu at (243.0, 113.4)
- added SW9: SW_Push, Button_Switch_Keyboard:SW_Cherry_MX_1.00u_PCB, F.Cu at (222.4, 234.1)
- added U3: 74HC595, 74HC595:SO16, F.Cu at (187.5, 99.3)
- J1: value Raspberry_Pi_4 -> Conn_01x01_Socket; footprint Connector_PinHeader_2.54mm:PinHeader_2x20_P2.54mm_Vertical -> Connector_PinHeader_2.54mm:PinHeader_1x01_P2.54mm_Vertical; moved to B.Cu
- R1: renamed from R2; moved to B.Cu
- R2: renamed from R1; moved to B.Cu
- U1: renamed from U3; moved to B.Cu
- U2: renamed from U1; moved to B.Cu
- moved U13 223.6 mm to (271.4, 31.7)
- moved U25 221.1 mm to (322.4, 126.1)
- moved U26 193.7 mm to (182.4, 247.1)
- moved U16 169.7 mm to (257.9, 31.7)
- moved U24 168.4 mm to (252.4, 126.1)
- moved U14 165.3 mm to (224.9, 31.7)
- moved U15 164.7 mm to (238.4, 31.7)
- moved U11 124.8 mm to (138.9, 31.7)
- moved U23 118.6 mm to (182.4, 126.1)
- moved R1 115.1 mm to (247.5, 53.0)
- moved U19 104.0 mm to (125.4, 31.7)
- moved U1 102.2 mm to (272.6, 72.6), turned to 90 degrees
- moved R2 96.3 mm to (93.8, 56.5), turned to 180 degrees
- moved U12 84.5 mm to (105.9, 31.7)
- moved U22 77.7 mm to (112.4, 126.1)
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Connections:
- J1 pad 1: Net-(J1-3V3-Pad1) -> Net-(J1-Pin_1)
- R1 pad 1: Net-(U1-V+) -> Net-(5V1-Pin_1)
- R2 pad 1: Net-(U1-V+) -> Net-(5V1-Pin_1)
- U1 pad 12: Net-(J1-~{CE1}_SPI0/GPIO07) -> Net-(MAXCS1-Pin_1)
- U1 pad 13: Net-(J1-SCLK_SPI0/GPIO11) -> Net-(M1-SCK)
- U1 pad 19: Net-(U1-V+) -> Net-(5V1-Pin_1)
- U1 pad 4: Net-(J1-GND-Pad14) -> Net-(GND1-Pin_1)
- U1 pad 5: /digit_max_1/DIG_7 -> /DIG_7
- U1 pad 8: /digit_max_1/DIG_6 -> /DIG_6
- U1 pad 9: Net-(J1-GND-Pad14) -> Net-(GND1-Pin_1)
- U2 pad 1: Net-(J1-MOSI_SPI0/GPIO10) -> Net-(M1-MOSI)
- U2 pad 12: Net-(J1-~{CE1}_SPI0/GPIO07) -> Net-(MAXCS1-Pin_1)
- U2 pad 13: Net-(J1-SCLK_SPI0/GPIO11) -> Net-(M1-SCK)
- U2 pad 19: Net-(U1-V+) -> Net-(5V1-Pin_1)
- U2 pad 4: Net-(J1-GND-Pad14) -> Net-(GND1-Pin_1)
- U2 pad 5: /digit_max_2/DIG_7 -> Net-(J3-Pin_1)
- U2 pad 8: /digit_max_2/DIG_6 -> Net-(J2-Pin_1)
- U2 pad 9: Net-(J1-GND-Pad14) -> Net-(GND1-Pin_1)
Routing:
- net Net-(3V1-Pin_1): track 0.00 -> 870.7 mm
- net Net-(GND1-Pin_1): track 0.00 -> 825.0 mm
- net Net-(J6-Pin_1): track 0.00 -> 461.8 mm
- net Net-(J4-Pin_1): track 0.00 -> 408.3 mm
- net Net-(J1-Pin_1): track 0.00 -> 268.8 mm
- net Net-(D2-A): track 0.00 -> 227.2 mm
- net Net-(5V1-Pin_1): track 0.00 -> 201.2 mm
- net Net-(D10-A): track 0.00 -> 117.0 mm
- net Net-(D13-A): track 0.00 -> 61.2 mm
- net Net-(D6-A): track 0.00 -> 57.9 mm
- net Net-(D12-A): track 0.00 -> 52.7 mm
- net Net-(D7-A): track 0.00 -> 42.6 mm
- net Net-(D1-A): track 0.00 -> 40.0 mm
- net Net-(D8-A): track 0.00 -> 34.3 mm
- net Net-(D11-A): track 0.00 -> 34.3 mm
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
Commit message: addicted to pla
Parts:
- removed U25, U26: SM420561N, Display_7Segment:7SegmentLED_LTS6760_LTS6780
- added U17: SM420561N, Display_7Segment:7SegmentLED_LTS6760_LTS6780, F.Cu at (322.4, 126.1)
- added U18: SM420561N, Display_7Segment:7SegmentLED_LTS6760_LTS6780, F.Cu at (182.4, 237.1)
- 3V1, 5V1, GND1, IRQ1, MAXCS1, MISO1, MOSI1, RST1, SCK1, SCS1: moved to F.Cu
- moved 3V1 97.2 mm to (106.4, 44.2), turned to 0 degrees
- moved IRQ1 95.9 mm to (111.0, 39.5), turned to 0 degrees
- moved MAXCS1 95.9 mm to (111.0, 44.1), turned to 0 degrees
- moved SCK1 95.9 mm to (111.0, 53.6), turned to 0 degrees
- moved SCS1 95.9 mm to (111.0, 58.2), turned to 0 degrees
- moved J2 94.5 mm to (156.5, 23.5)
- moved J3 94.5 mm to (163.5, 23.5)
- moved MISO1 93.4 mm to (106.4, 58.2), turned to 0 degrees
- moved RST1 90.3 mm to (111.0, 48.7), turned to 0 degrees
- moved MOSI1 86.8 mm to (106.4, 53.5), turned to 0 degrees
- moved GND1 63.9 mm to (106.4, 48.8), turned to 0 degrees
- moved R2 53.1 mm to (144.5, 40.5)
- moved U2 53.1 mm to (147.1, 56.3)
- moved 5V1 26.1 mm to (106.4, 39.5), turned to 0 degrees
- moved J1 10.3 mm to (178.5, 99.5)
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Connections:
- U1 pad 5: /DIG_7 -> /digit_max_1/DIG_7
- U1 pad 8: /DIG_6 -> /digit_max_1/DIG_6
Routing:
- net Net-(M1-SCK): track 0.00 -> 617.3 mm, vias 0 -> 3
- net /digit_max_1/SEG_G: track 0.00 -> 567.7 mm, vias 0 -> 3
- net /digit_max_1/SEG_C: track 0.00 -> 553.5 mm, vias 0 -> 2
- net /digit_max_1/SEG_E: track 0.00 -> 546.9 mm, vias 0 -> 3
- net /digit_max_1/SEG_D: track 0.00 -> 543.3 mm, vias 0 -> 4
- net /digit_max_1/SEG_F: track 0.00 -> 538.2 mm, vias 0 -> 3
- net Net-(IRQ1-Pin_1): track 0.00 -> 535.5 mm, vias 0 -> 2
- net Net-(M1-RST): track 0.00 -> 534.3 mm, vias 0 -> 2
- net /digit_max_1/SEG_B: track 0.00 -> 530.1 mm, vias 0 -> 3
- net /digit_max_1/SEG_DP: track 0.00 -> 527.5 mm, vias 0 -> 2
- net /digit_max_1/SEG_A: track 0.00 -> 526.7 mm, vias 0 -> 2
- net Net-(M1-MISO): track 0.00 -> 521.0 mm, vias 0 -> 1
- net Net-(M1-MOSI): track 0.00 -> 442.9 mm, vias 0 -> 3
- net /digit_max_2/SEG_C: track 0.00 -> 378.3 mm, vias 0 -> 2
- net /digit_max_2/SEG_DP: track 0.00 -> 370.4 mm, vias 0 -> 1
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Other:
- board outline added: 348 x 232.5 mm
