File: kicad/rpi-balatro/rpi-balatro.kicad_sch (KiCad schematic)
At the start: 13 parts, among them J1 Raspberry_Pi_4, J2 Conn_01x01_Socket, J3 Conn_01x01_Socket, U2 MAX7221xNG, U3 MAX7221xNG, U4 MAX7221xNG, U6 MAX7221xNG, U8 MAX7221xNG

Commit message: addicted to pla
Parts:
- added J10, J11, J4, J5, J6, J7, J8, J9: Conn_01x01_Socket, Connector_PinHeader_2.54mm:PinHeader_1x01_P2.54mm_Vertical, symbol Connector:Conn_01x01_Socket
- J2, J3: footprint (none) -> Connector_PinHeader_2.54mm:PinHeader_1x01_P2.54mm_Vertical
Connections:
- net digit_max_7/SEG_G: now reaches J3.1 (Pin_1)
- net digit_max_7/DIG_1: now reaches J2.1 (Pin_1)
- new net digit_max_7/DIG_0: J4.1 (Pin_1)
- new net digit_max_7/SEG_A: J11.1 (Pin_1)
- new net digit_max_7/SEG_B: J10.1 (Pin_1)
- new net digit_max_7/SEG_C: J8.1 (Pin_1)
- new net digit_max_7/SEG_D: J9.1 (Pin_1)
- new net digit_max_7/SEG_DP: J5.1 (Pin_1)
- new net digit_max_7/SEG_E: J7.1 (Pin_1)
- new net digit_max_7/SEG_F: J6.1 (Pin_1)
Other:
- added sheet digit_max_7 (dig_max_7.kicad_sch)
- moved on the sheet: J2, J3
